Commit message: Update MoveIt config and add floor publisher script
Expanded and updated RViz MoveIt configuration files, added new RViz config and backup files, and updated UR3 URDF joint orientation. Added new USD and JSON files for Isaac Sim, and introduced a Python script to publish a floor collision object to the PlanningScene.

File: skoltech/urdf/UR3_with_gripper.urdf (robot description, URDF)
Before this commit: robot ur3, 22 links, 21 joints
Joints:
- joint mount_gripper_to_tool0: origin xyz=0 0 0 rpy=1.5707 -1.5707 0 -> xyz=0 0 0 rpy=0 -1.5707 0
